Commit message: 粗さ情報のグリッド表示までできるようになった。

File: install/hesai_description/share/hesai_description/urdf/gazebo.urdf.xacro (robot description, xacro)
@@ -1,56 +1 @@
-<?xml version="1.0"?>
-<robot xmlns:xacro="http://www.ros.org/wiki/xacro">
-  <xacro:macro name="hesai_gazebo" params="prefix lidar_frame:=hesai_lidar topic_name=/hesai/pandar
-               min_range:=0.4 max_range:=80.0 min_horizontal_angle:=-180.0 max_horizontal_angle:=180.0
-               min_vertical_angle:=-16.0 max_vertical_angle:=15.0 hz:=10 samples:=2000 lasers:=32
-               collision_range:=0.3 noise:=0.008 visualize:=false use_gpu:=true">
-    <gazebo reference="${lidar_frame}">
-      <xacro:if value="${use_gpu}">
-        <xacro:property name="ray_type" value="gpu_ray" />
-        <xacro:property name="laser_plugin" value="libgazebo_ros_velodyne_gpu_laser.so" />
-      </xacro:if>
-      <xacro:unless value="${use_gpu}">
-        <xacro:property name="ray_type" value="ray" />
-        <xacro:property name="laser_plugin" value="libgazebo_ros_velodyne_laser.so" />
-      </xacro:unless>
-      <sensor type="${ray_type}" name="${prefix}hesai_sensor">
-        <pose>0 0 0 0 0 0</pose>
-        <visualize>${visualize}</visualize>
-        <update_rate>${hz}</update_rate>
-        <ray>
-          <scan>
-            <horizontal>
-              <samples>${samples}</samples>
-              <resolution>1</resolution>
-              <min_angle>${min_horizontal_angle*pi/180.0}</min_angle>
-              <max_angle>${max_horizontal_angle*pi/180.0}</max_angle>
-            </horizontal>
-            <vertical>
-              <samples>${lasers}</samples>
-              <resolution>1</resolution>
-              <min_angle>${min_vertical_angle*pi/180.0}</min_angle>
-              <max_angle>${max_vertical_angle*pi/180.0}</max_angle>
-            </vertical>
-          </scan>
-          <range>
-            <min>${collision_range}</min>
-            <max>${max_range+1}</max>
-            <resolution>0.001</resolution>
-          </range>
-          <noise>
-            <type>gaussian</type>
-            <mean>0.0</mean>
-            <stddev>0.0</stddev>
-          </noise>
-        </ray>
-        <plugin name="${prefix}gazebo_ros_laser_controller" filename="${laser_plugin}">
-          <topicName>${topic_name}</topicName>
-          <frameName>${lidar_frame}</frameName>
-          <min_range>${min_range}</min_range>
-          <max_range>${max_range}</max_range>
-          <gaussianNoise>${noise}</gaussianNoise>
-        </plugin>
-      </sensor>
-    </gazebo>
-  </xacro:macro>
-</robot>
+/home/takuto/scout_ws/src/hesai_description/urdf/gazebo.urdf.xacro

File: install/hesai_description/share/hesai_description/urdf/hesai_qt64.urdf.xacro (robot description, xacro)
@@ -1,47 +1 @@
-<?xml version="1.0"?>
-<robot name="hesai_qt64" xmlns:xacro="http://www.ros.org/wiki/xacro">
-  <xacro:macro name="hesai_qt64" params="parent *origin prefix:='' name:=pandar_qt64
-                                         topic_name:=/hesai/pandar
-                                         simulation:=false lidar_frame:=hesai_lidar use_gpu:=true">
-    <joint name="${parent}_to_${prefix}hesai" type="fixed">
-      <xacro:insert_block name="origin"/>
-      <parent link="${parent}" />
-      <child link="${prefix}hesai_base" />
-    </joint>
-    <link name="${prefix}hesai_base">
-      <visual>
-        <origin xyz="0 0 0" rpy="0 0 0" />
-        <geometry>
-          <mesh filename="package://hesai_description/meshes/visual/qt64.dae" />
-        </geometry>
-      </visual>
-      <inertial>
-        <!-- TODO Still correspond to values of XT32 -->
-        <origin xyz="-0.015e-3 0.0 37.494e-3" rpy="0 0 0" />
-        <mass value="0.807" />
-        <inertia ixx="886.81e-6" ixy="5.802e-11" ixz="-0.34e-6" iyy="898.12e-6" iyz="-0.014e-6" izz="1004.287e-6" />
-      </inertial>
-      <collision>
-        <origin xyz="0 0 38.0e-3"/>
-        <geometry>
-          <cylinder radius="51.500e-3" length="76.0e-3" />
-        </geometry>
-      </collision>
-    </link>
-    <link name="${lidar_frame}"/>
-    <joint name="${prefix}hesai_base_to_${lidar_frame}" type="fixed">
-      <!-- See page 12 of QT64 user manual -->
-      <!-- Note that the X axis points left See manual page 11 -->
-      <origin xyz="0.0 0.0 50.4e-3" rpy="0.0 0.0 ${pi/2}"/>
-      <parent link="${prefix}hesai_base"/>
-      <child link="${lidar_frame}" />
-    </joint>
-    <xacro:if value="${simulation}">
-      <xacro:include filename="$(find hesai_description)/urdf/gazebo.urdf.xacro"/>
-      <xacro:hesai_gazebo prefix="${prefix}" lidar_frame="${lidar_frame}" topic_name="${topic_name}" min_range="0.1" max_range="20.0"
-        min_horizontal_angle="-180.0" max_horizontal_angle="180.0" min_vertical_angle="-52.1" max_vertical_angle="52.1"
-        hz="10" samples="600" lasers="64" collision_range="0.3" noise="0.008" use_gpu="${use_gpu}"
-      />
-    </xacro:if>
-  </xacro:macro>
-</robot>
+/home/takuto/scout_ws/src/hesai_description/urdf/hesai_qt64.urdf.xacro

File: install/hesai_description/share/hesai_description/urdf/hesai_qt64_standalone.urdf.xacro (robot description, xacro)
@@ -1,12 +1 @@
-<?xml version="1.0"?>
-<robot name="hesai" xmlns:xacro="http://www.ros.org/wiki/xacro">
-  <xacro:arg name="prefix" default="" />
-  <xacro:arg name="simulation" default="false" />
-  <xacro:arg name="use_gpu" default="true" />
-  <xacro:include filename="$(find hesai_description)/urdf/hesai_qt64.urdf.xacro" />
-  <link name="base"/>
-  <xacro:hesai_qt64 parent="base" prefix="$(arg prefix)" lidar_frame="$(arg prefix)hesai_lidar"
-                    simulation="$(arg simulation)" use_gpu="$(arg use_gpu)" >
-    <origin xyz="0 0 0" rpy="0 0 0" />
-  </xacro:hesai_qt64>
-</robot>
+/home/takuto/scout_ws/src/hesai_description/urdf/hesai_qt64_standalone.urdf.xacro

File: install/hesai_description/share/hesai_description/urdf/hesai_xt32.urdf.xacro (robot description, xacro)
@@ -1,48 +1 @@
-<?xml version="1.0"?>
-<robot name="hesai_xt32" xmlns:xacro="http://www.ros.org/wiki/xacro">
-  <xacro:macro name="hesai_xt32" params="parent *origin prefix:='' name:=hesai_xt32
-                                        topic_name:=/hesai/pandar
-                                        simulation:=false lidar_frame:=hesai_lidar use_gpu:=true">
-    <joint name="${parent}_to_${prefix}hesai" type="fixed">
-      <xacro:insert_block name="origin"/>
-      <parent link="${parent}" />
-      <child link="${prefix}hesai_base" />
-    </joint>
-    <link name="${prefix}hesai_base">
-      <visual>
-        <origin xyz="0 0 0" rpy="0 0 0" />
-        <geometry>
-          <mesh filename="package://hesai_description/meshes/visual/xt32.dae" />
-        </geometry>
-      </visual>
-      <inertial>
-        <!-- Taken from CAD assuming constant density and mass 0.807 -->
-        <origin xyz="-0.015e-3 0.0 37.494e-3" rpy="0 0 0" />
-        <!-- Taken from datasheet -->
-        <mass value="0.807" />
-        <!-- Taken from CAD assuming constant density and mass 0.807 -->
-        <inertia ixx="886.81e-6" ixy="5.802e-11" ixz="-0.34e-6" iyy="898.12e-6" iyz="-0.014e-6" izz="1004.287e-6" />
-      </inertial>
-      <collision>
-        <origin xyz="0 0 38.0e-3"/>
-        <geometry>
-          <cylinder radius="51.500e-3" length="76.0e-3" />
-        </geometry>
-      </collision>
-    </link>
-    <link name="${lidar_frame}"/>
-    <joint name="${prefix}hesai_base_to_${lidar_frame}" type="fixed">
-      <!-- See XT32 user manual -->
-      <origin xyz="0.0 0.0 46.4e-3" rpy="0.0 0.0 ${pi/2}"/>
-      <parent link="${prefix}hesai_base"/>
-      <child link="${lidar_frame}" />
-    </joint>
-    <xacro:if value="${simulation}">
-      <xacro:include filename="$(find hesai_description)/urdf/gazebo.urdf.xacro"/>
-      <xacro:hesai_gazebo prefix="${prefix}" lidar_frame="${lidar_frame}" topic_name="${topic_name}" min_range="0.4" max_range="80.0"
-        min_horizontal_angle="-180.0" max_horizontal_angle="180.0" min_vertical_angle="-16.0" max_vertical_angle="15.0"
-        hz="10" samples="2000" lasers="32" collision_range="0.3" noise="0.008" use_gpu="${use_gpu}"
-      />
-    </xacro:if>
-  </xacro:macro>
-</robot>
+/home/takuto/scout_ws/src/hesai_description/urdf/hesai_xt32.urdf.xacro

File: install/hesai_description/share/hesai_description/urdf/hesai_xt32_standalone.urdf.xacro (robot description, xacro)
@@ -1,12 +1 @@
-<?xml version="1.0"?>
-<robot name="hesai" xmlns:xacro="http://www.ros.org/wiki/xacro">
-  <xacro:arg name="prefix" default="" />
-  <xacro:arg name="simulation" default="false" />
-  <xacro:arg name="use_gpu" default="true" />
-  <xacro:include filename="$(find hesai_description)/urdf/hesai_xt32.urdf.xacro" />
-  <link name="base"/>
-  <xacro:hesai_xt32 parent="base" prefix="$(arg prefix)" lidar_frame="$(arg prefix)hesai_lidar"
-                    simulation="$(arg simulation)" use_gpu="$(arg use_gpu)" >
-    <origin xyz="0 0 0" rpy="0 0 0" />
-  </xacro:hesai_xt32>
-</robot>
+/home/takuto/scout_ws/src/hesai_description/urdf/hesai_xt32_standalone.urdf.xacro

Commit message: エラーなく一旦

File: install/hesai_description/share/hesai_description/urdf/gazebo.urdf.xacro (robot description, xacro)
@@ -1 +1,56 @@
-/home/takuto/scout_ws/src/hesai_description/urdf/gazebo.urdf.xacro
+<?xml version="1.0"?>
+<robot xmlns:xacro="http://www.ros.org/wiki/xacro">
+  <xacro:macro name="hesai_gazebo" params="prefix lidar_frame:=hesai_lidar topic_name=/hesai/pandar
+               min_range:=0.4 max_range:=80.0 min_horizontal_angle:=-180.0 max_horizontal_angle:=180.0
+               min_vertical_angle:=-16.0 max_vertical_angle:=15.0 hz:=10 samples:=2000 lasers:=32
+               collision_range:=0.3 noise:=0.008 visualize:=false use_gpu:=true">
+    <gazebo reference="${lidar_frame}">
+      <xacro:if value="${use_gpu}">
+        <xacro:property name="ray_type" value="gpu_ray" />
+        <xacro:property name="laser_plugin" value="libgazebo_ros_velodyne_gpu_laser.so" />
+      </xacro:if>
+      <xacro:unless value="${use_gpu}">
+        <xacro:property name="ray_type" value="ray" />
+        <xacro:property name="laser_plugin" value="libgazebo_ros_velodyne_laser.so" />
+      </xacro:unless>
+      <sensor type="${ray_type}" name="${prefix}hesai_sensor">
+        <pose>0 0 0 0 0 0</pose>
+        <visualize>${visualize}</visualize>
+        <update_rate>${hz}</update_rate>
+        <ray>
+          <scan>
+            <horizontal>
+              <samples>${samples}</samples>
+              <resolution>1</resolution>
+              <min_angle>${min_horizontal_angle*pi/180.0}</min_angle>
+              <max_angle>${max_horizontal_angle*pi/180.0}</max_angle>
+            </horizontal>
+            <vertical>
+              <samples>${lasers}</samples>
+              <resolution>1</resolution>
+              <min_angle>${min_vertical_angle*pi/180.0}</min_angle>
+              <max_angle>${max_vertical_angle*pi/180.0}</max_angle>
+            </vertical>
+          </scan>
+          <range>
+            <min>${collision_range}</min>
+            <max>${max_range+1}</max>
+            <resolution>0.001</resolution>
+          </range>
+          <noise>
+            <type>gaussian</type>
+            <mean>0.0</mean>
+            <stddev>0.0</stddev>
+          </noise>
+        </ray>
+        <plugin name="${prefix}gazebo_ros_laser_controller" filename="${laser_plugin}">
+          <topicName>${topic_name}</topicName>
+          <frameName>${lidar_frame}</frameName>
+          <min_range>${min_range}</min_range>
+          <max_range>${max_range}</max_range>
+          <gaussianNoise>${noise}</gaussianNoise>
+        </plugin>
+      </sensor>
+    </gazebo>
+  </xacro:macro>
+</robot>

File: install/hesai_description/share/hesai_description/urdf/hesai_qt64.urdf.xacro (robot description, xacro)
@@ -1 +1,47 @@
-/home/takuto/scout_ws/src/hesai_description/urdf/hesai_qt64.urdf.xacro
+<?xml version="1.0"?>
+<robot name="hesai_qt64" xmlns:xacro="http://www.ros.org/wiki/xacro">
+  <xacro:macro name="hesai_qt64" params="parent *origin prefix:='' name:=pandar_qt64
+                                         topic_name:=/hesai/pandar
+                                         simulation:=false lidar_frame:=hesai_lidar use_gpu:=true">
+    <joint name="${parent}_to_${prefix}hesai" type="fixed">
+      <xacro:insert_block name="origin"/>
+      <parent link="${parent}" />
+      <child link="${prefix}hesai_base" />
+    </joint>
+    <link name="${prefix}hesai_base">
+      <visual>
+        <origin xyz="0 0 0" rpy="0 0 0" />
+        <geometry>
+          <mesh filename="package://hesai_description/meshes/visual/qt64.dae" />
+        </geometry>
+      </visual>
+      <inertial>
+        <!-- TODO Still correspond to values of XT32 -->
+        <origin xyz="-0.015e-3 0.0 37.494e-3" rpy="0 0 0" />
+        <mass value="0.807" />
+        <inertia ixx="886.81e-6" ixy="5.802e-11" ixz="-0.34e-6" iyy="898.12e-6" iyz="-0.014e-6" izz="1004.287e-6" />
+      </inertial>
+      <collision>
+        <origin xyz="0 0 38.0e-3"/>
+        <geometry>
+          <cylinder radius="51.500e-3" length="76.0e-3" />
+        </geometry>
+      </collision>
+    </link>
+    <link name="${lidar_frame}"/>
+    <joint name="${prefix}hesai_base_to_${lidar_frame}" type="fixed">
+      <!-- See page 12 of QT64 user manual -->
+      <!-- Note that the X axis points left See manual page 11 -->
+      <origin xyz="0.0 0.0 50.4e-3" rpy="0.0 0.0 ${pi/2}"/>
+      <parent link="${prefix}hesai_base"/>
+      <child link="${lidar_frame}" />
+    </joint>
+    <xacro:if value="${simulation}">
+      <xacro:include filename="$(find hesai_description)/urdf/gazebo.urdf.xacro"/>
+      <xacro:hesai_gazebo prefix="${prefix}" lidar_frame="${lidar_frame}" topic_name="${topic_name}" min_range="0.1" max_range="20.0"
+        min_horizontal_angle="-180.0" max_horizontal_angle="180.0" min_vertical_angle="-52.1" max_vertical_angle="52.1"
+        hz="10" samples="600" lasers="64" collision_range="0.3" noise="0.008" use_gpu="${use_gpu}"
+      />
+    </xacro:if>
+  </xacro:macro>
+</robot>

File: install/hesai_description/share/hesai_description/urdf/hesai_qt64_standalone.urdf.xacro (robot description, xacro)
@@ -1 +1,12 @@
-/home/takuto/scout_ws/src/hesai_description/urdf/hesai_qt64_standalone.urdf.xacro
+<?xml version="1.0"?>
+<robot name="hesai" xmlns:xacro="http://www.ros.org/wiki/xacro">
+  <xacro:arg name="prefix" default="" />
+  <xacro:arg name="simulation" default="false" />
+  <xacro:arg name="use_gpu" default="true" />
+  <xacro:include filename="$(find hesai_description)/urdf/hesai_qt64.urdf.xacro" />
+  <link name="base"/>
+  <xacro:hesai_qt64 parent="base" prefix="$(arg prefix)" lidar_frame="$(arg prefix)hesai_lidar"
+                    simulation="$(arg simulation)" use_gpu="$(arg use_gpu)" >
+    <origin xyz="0 0 0" rpy="0 0 0" />
+  </xacro:hesai_qt64>
+</robot>

File: install/hesai_description/share/hesai_description/urdf/hesai_xt32.urdf.xacro (robot description, xacro)
@@ -1 +1,48 @@
-/home/takuto/scout_ws/src/hesai_description/urdf/hesai_xt32.urdf.xacro
+<?xml version="1.0"?>
+<robot name="hesai_xt32" xmlns:xacro="http://www.ros.org/wiki/xacro">
+  <xacro:macro name="hesai_xt32" params="parent *origin prefix:='' name:=hesai_xt32
+                                        topic_name:=/hesai/pandar
+                                        simulation:=false lidar_frame:=hesai_lidar use_gpu:=true">
+    <joint name="${parent}_to_${prefix}hesai" type="fixed">
+      <xacro:insert_block name="origin"/>
+      <parent link="${parent}" />
+      <child link="${prefix}hesai_base" />
+    </joint>
+    <link name="${prefix}hesai_base">
+      <visual>
+        <origin xyz="0 0 0" rpy="0 0 0" />
+        <geometry>
+          <mesh filename="package://hesai_description/meshes/visual/xt32.dae" />
+        </geometry>
+      </visual>
+      <inertial>
+        <!-- Taken from CAD assuming constant density and mass 0.807 -->
+        <origin xyz="-0.015e-3 0.0 37.494e-3" rpy="0 0 0" />
+        <!-- Taken from datasheet -->
+        <mass value="0.807" />
+        <!-- Taken from CAD assuming constant density and mass 0.807 -->
+        <inertia ixx="886.81e-6" ixy="5.802e-11" ixz="-0.34e-6" iyy="898.12e-6" iyz="-0.014e-6" izz="1004.287e-6" />
+      </inertial>
+      <collision>
+        <origin xyz="0 0 38.0e-3"/>
+        <geometry>
+          <cylinder radius="51.500e-3" length="76.0e-3" />
+        </geometry>
+      </collision>
+    </link>
+    <link name="${lidar_frame}"/>
+    <joint name="${prefix}hesai_base_to_${lidar_frame}" type="fixed">
+      <!-- See XT32 user manual -->
+      <origin xyz="0.0 0.0 46.4e-3" rpy="0.0 0.0 ${pi/2}"/>
+      <parent link="${prefix}hesai_base"/>
+      <child link="${lidar_frame}" />
+    </joint>
+    <xacro:if value="${simulation}">
+      <xacro:include filename="$(find hesai_description)/urdf/gazebo.urdf.xacro"/>
+      <xacro:hesai_gazebo prefix="${prefix}" lidar_frame="${lidar_frame}" topic_name="${topic_name}" min_range="0.4" max_range="80.0"
+        min_horizontal_angle="-180.0" max_horizontal_angle="180.0" min_vertical_angle="-16.0" max_vertical_angle="15.0"
+        hz="10" samples="2000" lasers="32" collision_range="0.3" noise="0.008" use_gpu="${use_gpu}"
+      />
+    </xacro:if>
+  </xacro:macro>
+</robot>

File: install/hesai_description/share/hesai_description/urdf/hesai_xt32_standalone.urdf.xacro (robot description, xacro)
@@ -1 +1,12 @@
-/home/takuto/scout_ws/src/hesai_description/urdf/hesai_xt32_standalone.urdf.xacro
+<?xml version="1.0"?>
+<robot name="hesai" xmlns:xacro="http://www.ros.org/wiki/xacro">
+  <xacro:arg name="prefix" default="" />
+  <xacro:arg name="simulation" default="false" />
+  <xacro:arg name="use_gpu" default="true" />
+  <xacro:include filename="$(find hesai_description)/urdf/hesai_xt32.urdf.xacro" />
+  <link name="base"/>
+  <xacro:hesai_xt32 parent="base" prefix="$(arg prefix)" lidar_frame="$(arg prefix)hesai_lidar"
+                    simulation="$(arg simulation)" use_gpu="$(arg use_gpu)" >
+    <origin xyz="0 0 0" rpy="0 0 0" />
+  </xacro:hesai_xt32>
+</robot>
